Commit message: Working laserscan and joints world added

File: install/ball_follower/share/ball_follower/description/robot.urdf.xacro (robot description, xacro)
@@ -2,3 +2,6 @@
 <robot xmlns:xacro="http://www.ros.org/wiki/xacro"  name="robot">
     <xacro:include filename="robot_core.xacro" />
+    <xacro:include filename="gazebo_control.xacro" />
+    <xacro:include filename="lidar.xacro" />
+    <xacro:include filename="camera.xacro" />
 </robot>

File: install/ball_follower/share/ball_follower/description/robot_core.xacro (robot description, xacro)
@@ -10,15 +10,23 @@
     <xacro:property name="chassis_y" value="0.8" />
     <xacro:property name="chassis_z" value="0.5" />
-    <xacro:property name="chassis_h" value="0.1" />
+    <xacro:property name="chassis_h" value="0.2" />
     <xacro:property name="wheel_l" value="0.1" />
-    <xacro:property name="wheel_r" value="0.1" />
-    <xacro:property name="caster_r" value="0.1" />
+    <xacro:property name="wheel_r" value="0.2" />
+    <xacro:property name="caster_r" value="0.2" />
     <xacro:property name="fork_x" value="0.6" />
     <xacro:property name="fork_y" value="0.7" />
     <xacro:property name="fork_z" value="0.05" />
-    <xacro:property name="fork_h" value="0.1" />
+    <xacro:property name="fork_h" value="0.2" />
     <!-- BASE LINK -->
     <link name="base_link">
     </link>
+    <!-- BASE FOOTPRINT LINK -->
+    <link name="base_footprint">
+    </link>
+    <joint name="base_footprint_joint" type="fixed">
+        <parent link="base_link"/>
+        <child link="base_footprint"/>
+        <origin xyz="0.0 0.0 0.0" rpy="0.0 0.0 0.0"/>
+    </joint>
     <!-- CHASSIS LINK -->
     <joint name="chassis_joint" type="fixed">
@@ -52,9 +60,9 @@
     </link>
     <!-- LEFT WHEEL LINK -->
-    <joint name="left_wheel_joint" type="fixed">
-        <parent link="chassis"/>
+    <joint name="left_wheel_joint" type="continuous">
+        <parent link="base_link"/>
         <child link="left_wheel"/>
         <origin xyz="${-chassis_x/5} ${chassis_y/2+wheel_l/2} ${wheel_r-chassis_h-chassis_z/2}" rpy="-1.5707 0.0 0.0"/>
-        <!-- <axis xyz="0 0 1"/> -->
+        <axis xyz="0 0 1"/>
     </joint>
         <!-- LINK -->
@@ -83,13 +91,13 @@
     </link>
     <!-- RIGHT WHEEL LINK -->
-    <joint name="right_wheel_joint" type="fixed">
-        <parent link="chassis"/>
+    <joint name="right_wheel_joint" type="continuous">
+        <parent link="base_link"/>
         <child link="right_wheel"/>
         <origin xyz="${-chassis_x/5} ${-chassis_y/2-wheel_l/2} ${wheel_r-chassis_h-chassis_z/2}" rpy="-1.5707 0.0 0.0"/>
-        <!-- <axis xyz="0 0 -1"/> -->
+        <axis xyz="0 0 -1"/>
     </joint>
         <!-- LINK -->
     <link name="right_wheel">
-        <xacro:inertial_cylinder mass="15" radius="${wheel_r}" length="${wheel_l}">
+        <xacro:inertial_cylinder mass="${wheel_m}" radius="${wheel_r}" length="${wheel_l}">
             <origin xyz="0.0 0 0" rpy="0 0 0"/>
         </xacro:inertial_cylinder>
@@ -121,5 +129,5 @@
         <!-- LINK -->
     <link name="caster">
-        <xacro:inertial_sphere mass="15" radius="0.1">
+        <xacro:inertial_sphere mass="${caster_m}" radius="${caster_r}">
             <origin xyz="0.0 0.0 0" rpy="0 0 0"/>
         </xacro:inertial_sphere>
@@ -182,15 +190,11 @@
         <material>Gazebo/Red</material>
     </gazebo>
+    <gazebo reference="fork">
+        <material>Gazebo/Grey</material>
+    </gazebo>
     <gazebo reference="caster">
         <material>Gazebo/Black</material>
-    </gazebo>
-    <gazebo reference="fork">
-        <material>Gazebo/Grey</material>
-    </gazebo>
-    <!-- <xacro:inertial_cylinder mass="15" length="20" radius="3">
-        <origin xyz="0.0 0.0 0.0" rpy="0 0 0">
-    </inertial_box>
-    <xacro:inertial_sphere mass="15" radius="8">
-        <origin xyz="0.0 0.0 0.0" rpy="0 0 0">
-    </inertial_box>-->
+        <mu1 value="0.001"/>
+        <mu2 value="0.001"/>
+    </gazebo>
 </robot>

File: src/bot/description/robot_core.xacro (robot description, xacro)
@@ -10,15 +10,23 @@
     <xacro:property name="chassis_y" value="0.8" />
     <xacro:property name="chassis_z" value="0.5" />
-    <xacro:property name="chassis_h" value="0.1" />
+    <xacro:property name="chassis_h" value="0.2" />
     <xacro:property name="wheel_l" value="0.1" />
-    <xacro:property name="wheel_r" value="0.1" />
-    <xacro:property name="caster_r" value="0.1" />
+    <xacro:property name="wheel_r" value="0.2" />
+    <xacro:property name="caster_r" value="0.2" />
     <xacro:property name="fork_x" value="0.6" />
     <xacro:property name="fork_y" value="0.7" />
     <xacro:property name="fork_z" value="0.05" />
-    <xacro:property name="fork_h" value="0.1" />
+    <xacro:property name="fork_h" value="0.2" />
     <!-- BASE LINK -->
     <link name="base_link">
     </link>
+    <!-- BASE FOOTPRINT LINK -->
+    <link name="base_footprint">
+    </link>
+    <joint name="base_footprint_joint" type="fixed">
+        <parent link="base_link"/>
+        <child link="base_footprint"/>
+        <origin xyz="0.0 0.0 0.0" rpy="0.0 0.0 0.0"/>
+    </joint>
     <!-- CHASSIS LINK -->
     <joint name="chassis_joint" type="fixed">
@@ -52,9 +60,9 @@
     </link>
     <!-- LEFT WHEEL LINK -->
-    <joint name="left_wheel_joint" type="fixed">
-        <parent link="chassis"/>
+    <joint name="left_wheel_joint" type="continuous">
+        <parent link="base_link"/>
         <child link="left_wheel"/>
         <origin xyz="${-chassis_x/5} ${chassis_y/2+wheel_l/2} ${wheel_r-chassis_h-chassis_z/2}" rpy="-1.5707 0.0 0.0"/>
-        <!-- <axis xyz="0 0 1"/> -->
+        <axis xyz="0 0 1"/>
     </joint>
         <!-- LINK -->
@@ -83,13 +91,13 @@
     </link>
     <!-- RIGHT WHEEL LINK -->
-    <joint name="right_wheel_joint" type="fixed">
-        <parent link="chassis"/>
+    <joint name="right_wheel_joint" type="continuous">
+        <parent link="base_link"/>
         <child link="right_wheel"/>
         <origin xyz="${-chassis_x/5} ${-chassis_y/2-wheel_l/2} ${wheel_r-chassis_h-chassis_z/2}" rpy="-1.5707 0.0 0.0"/>
-        <!-- <axis xyz="0 0 -1"/> -->
+        <axis xyz="0 0 -1"/>
     </joint>
         <!-- LINK -->
     <link name="right_wheel">
-        <xacro:inertial_cylinder mass="15" radius="${wheel_r}" length="${wheel_l}">
+        <xacro:inertial_cylinder mass="${wheel_m}" radius="${wheel_r}" length="${wheel_l}">
             <origin xyz="0.0 0 0" rpy="0 0 0"/>
         </xacro:inertial_cylinder>
@@ -121,5 +129,5 @@
         <!-- LINK -->
     <link name="caster">
-        <xacro:inertial_sphere mass="15" radius="0.1">
+        <xacro:inertial_sphere mass="${caster_m}" radius="${caster_r}">
             <origin xyz="0.0 0.0 0" rpy="0 0 0"/>
         </xacro:inertial_sphere>
@@ -182,9 +190,11 @@
         <material>Gazebo/Red</material>
     </gazebo>
+    <gazebo reference="fork">
+        <material>Gazebo/Grey</material>
+    </gazebo>
     <gazebo reference="caster">
         <material>Gazebo/Black</material>
-    </gazebo>
-    <gazebo reference="fork">
-        <material>Gazebo/Grey</material>
+        <mu1 value="0.001"/>
+        <mu2 value="0.001"/>
     </gazebo>
 </robot>
