Commit message: Images added in README

File: install/ball_follower/share/ball_follower/description/camera.xacro (robot description, xacro)
@@ -1,55 +1 @@
-<?xml version="1.0"?>
-<robot xmlns:xacro="http://www.ros.org/wiki/xacro"  name="robot">
-    <xacro:property name="camera_m" value="0.2" />
-    <xacro:property name="camera_x" value="0.05" />
-    <xacro:property name="camera_y" value="0.1" />
-    <xacro:property name="camera_z" value="0.02" />
-    <joint name="camera_joint" type="fixed">
-        <parent link="chassis"/>
-        <child link="camera_frame"/>
-        <origin xyz="${chassis_x/2} 0 ${chassis_h+3*camera_z}" rpy="0 0 0"/>
-    </joint>
-    <link name="camera_frame">
-        <xacro:inertial_box mass="${camera_m}" x="${camera_x}" y="${camera_y}" z="${camera_z}">
-            <origin xyz="0.0 0.0 0" rpy="0 0 0"/>
-        </xacro:inertial_box>
-        <visual>
-            <origin xyz="0.0 0.0 0.0" rpy="0 0 0"/>
-            <geometry>
-                <box size="${camera_x} ${camera_y} ${camera_z}"/>
-            </geometry>
-            <material name="red">
-                <color rgba="1 0 0 1"/>
-            </material>
-        </visual>
-        <collision>
-            <origin xyz="0.0 0.0 0.0" rpy="0 0 0"/>
-            <geometry>
-                <box size="${camera_x} ${camera_y} ${camera_z}"/>
-            </geometry>
-        </collision>
-    </link>
-    <gazebo reference="camera_frame">
-        <material>Gazebo/Black</material>
-        <sensor name="camera" type="camera">
-            <pose> 0 0 0 0 0 0 </pose>
-            <visualize>true</visualize>
-            <update_rate>10</update_rate>
-            <camera>
-                <horizontal_fov>1.089</horizontal_fov>
-                <image>
-                    <format>R8G8B8</format>
-                    <width>640</width>
-                    <height>480</height>
-                </image>
-                <clip>
-                    <near>0.05</near>
-                    <far>8.0</far>
-                </clip>
-            </camera>
-            <plugin name="camera_controller" filename="libgazebo_ros_camera.so">
-                <frame_name>camera_frame</frame_name>
-            </plugin>
-        </sensor>
-    </gazebo>
-</robot>
+/home/kuljot/Project/ball_follower/src/bot/description/camera.xacro

File: install/ball_follower/share/ball_follower/description/gazebo_control.xacro (robot description, xacro)
@@ -1,21 +1 @@
-<?xml version="1.0"?>
-<robot xmlns:xacro="http://www.ros.org/wiki/xacro">
-    <gazebo>
-        <plugin name="diff_drive" filename="libgazebo_ros_diff_drive.so">
-            <!-- WHEEL INFORMATION -->
-            <left_joint>left_wheel_joint</left_joint>
-            <right_joint>right_wheel_joint</right_joint>
-            <wheel_separation>0.9</wheel_separation>
-            <wheel_diameter>0.2</wheel_diameter>
-            <!-- LIMITS -->
-            <max_wheel_torque>200</max_wheel_torque>
-            <max_wheel_acceleration>10.0</max_wheel_acceleration>
-            <!-- OUTPUT -->
-            <odometry_frame>odom</odometry_frame>
-            <robot_base_frame>base_link</robot_base_frame>
-            <publish_odom>true</publish_odom>
-            <publish_odom_tf>true</publish_odom_tf>
-            <publish_wheel_tf>true</publish_wheel_tf>
-        </plugin>
-    </gazebo>
-</robot>
+/home/kuljot/Project/ball_follower/src/bot/description/gazebo_control.xacro

File: install/ball_follower/share/ball_follower/description/inertial_macros.xacro (robot description, xacro)
@@ -1,32 +1 @@
-<?xml version="1.0"?>
-<robot xmlns:xacro="http://www.ros.org/wiki/xacro" >
-    <!-- Specify some standard inertial calculations https://en.wikipedia.org/wiki/List_of_moments_of_inertia -->
-    <!-- These make use of xacro's mathematical functionality -->
-    <xacro:macro name="inertial_box" params="mass x y z *origin">
-        <inertial>
-            <xacro:insert_block name="origin"/>
-            <mass value="${mass}"/>
-            <inertia ixx="${(1/12) * mass * (y*y+z*z)}" ixy="0.0" ixz="0.0"
-                    iyy="${(1/12) * mass * (x*x+z*z)}" iyz="0.0"
-                    izz="${(1/12) * mass * (x*x+y*y)}" />
-        </inertial>
-    </xacro:macro>
-    <xacro:macro name="inertial_cylinder" params="mass length radius *origin">
-        <inertial>
-            <xacro:insert_block name="origin"/>
-            <mass value="${mass}"/>
-            <inertia ixx="${(1/2) * mass * (radius*radius)}" ixy="0.0" ixz="0.0"
-                    iyy="${mass * ((1/12) * (length*length) + (1/4) * (radius*radius))}" iyz="0.0"
-                    izz="${mass * ((1/12) * (length*length) + (1/4) * (radius*radius))}" />
-        </inertial>
-    </xacro:macro>
-    <xacro:macro name="inertial_sphere" params="mass radius *origin">
-        <inertial>
-            <xacro:insert_block name="origin"/>
-            <mass value="${mass}"/>
-            <inertia ixx="${(2/5) * mass * (radius*radius)}" ixy="0.0" ixz="0.0"
-                    iyy="${(2/5) * mass * (radius*radius)}" iyz="0.0"
-                    izz="${(2/5) * mass * (radius*radius)}" />
-        </inertial>
-    </xacro:macro>
-</robot>
+/home/kuljot/Project/ball_follower/src/bot/description/inertial_macros.xacro

File: install/ball_follower/share/ball_follower/description/lidar.xacro (robot description, xacro)
@@ -1,64 +1 @@
-<?xml version="1.0"?>
-<robot xmlns:xacro="http://www.ros.org/wiki/xacro"  name="robot">
-    <xacro:property name="laser_m" value="0.2" />
-    <xacro:property name="laser_r" value="0.05" />
-    <xacro:property name="laser_l" value="0.05" />
-    <joint name="laser_joint" type="fixed">
-        <parent link="chassis"/>
-        <child link="laser_frame"/>
-        <origin xyz="0 0 ${chassis_h+1.5*laser_l}" rpy="0 0 0"/>
-    </joint>
-    <link name="laser_frame">
-        <xacro:inertial_cylinder mass="${laser_m}" radius="${laser_r}" length="${laser_l}">
-            <origin xyz="0.0 0.0 0" rpy="0 0 0"/>
-        </xacro:inertial_cylinder>
-        <visual>
-            <origin xyz="0.0 0.0 0.0" rpy="0 0 0"/>
-            <geometry>
-                <cylinder radius="${laser_r}" length="${laser_l}"/>
-            </geometry>
-            <material name="red">
-                <color rgba="1 0 0 1"/>
-            </material>
-        </visual>
-        <collision>
-            <origin xyz="0.0 0.0 0.0" rpy="0 0 0"/>
-            <geometry>
-                <cylinder radius="${laser_r}" length="${laser_l}"/>
-            </geometry>
-        </collision>
-    </link>
-    <gazebo reference="laser_frame">
-        <material>Gazebo/Red</material>
-        <sensor name="laser" type="ray">
-            <pose> 0 0 0 0 0 0 </pose>
-            <visualize>true</visualize>
-            <update_rate>10</update_rate>
-            <ray>
-                <scan>
-                    <!-- <material>Gazebo/Red</material> -->
-                    <horizontal>
-                        <samples>360</samples>
-                        <min_angle>-3.14</min_angle>
-                        <max_angle>3.14</max_angle>
-                    </horizontal>
-                </scan>
-                <range>
-                    <min>0.3</min>
-                    <max>12</max>
-                </range>
-            </ray>
-            <plugin name="laser_controller" filename="libgazebo_ros_ray_sensor.so">
-                <ros>
-                    <!-- Scan can be seen at /laser_controller/out instead of /scan -->
-                    <!-- <argument>-ros-args -remap ~/out:=/scan</argument> -->
-                    <!-- <remapping>~/out:=/scan</remapping> -->
-                    <!-- <namespace>/</namespace> -->
-                    <argument>~/out:=scan</argument>
-                </ros>
-                <output_type>sensor_msgs/LaserScan</output_type>
-                <frame_name>laser_frame</frame_name>
-            </plugin>
-        </sensor>
-    </gazebo>
-</robot>
+/home/kuljot/Project/ball_follower/src/bot/description/lidar.xacro

File: install/ball_follower/share/ball_follower/description/robot.urdf.xacro (robot description, xacro)
@@ -1,7 +1 @@
-<?xml version="1.0"?>
-<robot xmlns:xacro="http://www.ros.org/wiki/xacro"  name="robot">
-    <xacro:include filename="robot_core.xacro" />
-    <xacro:include filename="gazebo_control.xacro" />
-    <xacro:include filename="lidar.xacro" />
-    <xacro:include filename="camera.xacro" />
-</robot>
+/home/kuljot/Project/ball_follower/src/bot/description/robot.urdf.xacro

File: install/ball_follower/share/ball_follower/description/robot_core.xacro (robot description, xacro)
@@ -1,200 +1 @@
-<?xml version="1.0"?>
-<robot xmlns:xacro="http://www.ros.org/wiki/xacro">
-    <xacro:include filename="inertial_macros.xacro" />
-    <!-- <xacro:include filename="visual_macros.xacro" /> -->
-    <xacro:property name="chassis_m" value="20" />
-    <xacro:property name="wheel_m" value="4" />
-    <xacro:property name="caster_m" value="4" />
-    <xacro:property name="fork_m" value="5" />
-    <xacro:property name="chassis_x" value="1" />
-    <xacro:property name="chassis_y" value="0.8" />
-    <xacro:property name="chassis_z" value="0.5" />
-    <xacro:property name="chassis_h" value="0.2" />
-    <xacro:property name="wheel_l" value="0.1" />
-    <xacro:property name="wheel_r" value="0.2" />
-    <xacro:property name="caster_r" value="0.2" />
-    <xacro:property name="fork_x" value="0.6" />
-    <xacro:property name="fork_y" value="0.7" />
-    <xacro:property name="fork_z" value="0.05" />
-    <xacro:property name="fork_h" value="0.2" />
-    <!-- BASE LINK -->
-    <link name="base_link">
-    </link>
-    <!-- BASE FOOTPRINT LINK -->
-    <link name="base_footprint">
-    </link>
-    <joint name="base_footprint_joint" type="fixed">
-        <parent link="base_link"/>
-        <child link="base_footprint"/>
-        <origin xyz="0.0 0.0 0.0" rpy="0.0 0.0 0.0"/>
-    </joint>
-    <!-- CHASSIS LINK -->
-    <joint name="chassis_joint" type="fixed">
-        <parent link="base_link"/>
-        <child link="chassis"/>
-        <origin xyz="0.0 0.0 ${chassis_z/2+wheel_r}" rpy="0.0 0.0 0.0"/>
-    </joint>
-        <!-- LINK -->
-    <link name="chassis">
-        <xacro:inertial_box mass="${chassis_m}" x="${chassis_x}" y="${chassis_y}" z="${chassis_z}">
-            <origin xyz="0 0.0 0" rpy="0 0 0"/>
-        </xacro:inertial_box>
-        <!-- <xacro:visual_box  x="1" y="0.5" z="0.5" r="0" g="1" b="0" a="1">
-            <origin xyz="0.2 0.0 0.35  " rpy="0 0 0"/>
-        </xacro:visual_box> -->
-        <visual>
-            <origin xyz="0.0 0.0 0" rpy="0 0 0"/>
-            <geometry>
-                <box size="${chassis_x} ${chassis_y} ${chassis_z}"/>
-            </geometry>
-            <material name="green">
-                <color rgba="0.175 0.93 0.93 1"/>
-            </material>
-        </visual>
-        <collision>
-            <origin xyz="0.0 0.0 0" rpy="0 0 0"/>
-            <geometry>
-                <box size="${chassis_x} ${chassis_y} ${chassis_z}"/>
-            </geometry>
-        </collision>
-    </link>
-    <!-- LEFT WHEEL LINK -->
-    <joint name="left_wheel_joint" type="continuous">
-        <parent link="base_link"/>
-        <child link="left_wheel"/>
-        <origin xyz="${-chassis_x/5} ${chassis_y/2+wheel_l/2} ${wheel_r-chassis_h-chassis_z/2}" rpy="-1.5707 0.0 0.0"/>
-        <axis xyz="0 0 1"/>
-    </joint>
-        <!-- LINK -->
-    <link name="left_wheel">
-        <xacro:inertial_cylinder mass="${wheel_m}" radius="${wheel_r}" length="${wheel_l}">
-            <origin xyz="0.0 0.0 0" rpy="0 0 0"/>
-        </xacro:inertial_cylinder>
-        <!-- <xacro:visual_cylinder radius="0.1" length="0.1" r="1.0" g="0" b="0" a="1">
-            <origin xyz="0.0 0.3 0.1" rpy="-1.5707 0 0"/>
-        </xacro:visual_cylinder> -->
-        <visual>
-            <origin xyz="0.0 0.0 0.0" rpy="0 0 0"/>
-            <geometry>
-                <cylinder radius="${wheel_r}" length="${wheel_l}"/>
-            </geometry>
-            <material name="red">
-                <color rgba="1 0 0 1"/>
-            </material>
-        </visual>
-        <collision>
-            <origin xyz="0.0 0.0 0.0" rpy="0 0 0"/>
-            <geometry>
-                <cylinder radius="${wheel_r}" length="${wheel_l}"/>
-            </geometry>
-        </collision>
-    </link>
-    <!-- RIGHT WHEEL LINK -->
-    <joint name="right_wheel_joint" type="continuous">
-        <parent link="base_link"/>
-        <child link="right_wheel"/>
-        <origin xyz="${-chassis_x/5} ${-chassis_y/2-wheel_l/2} ${wheel_r-chassis_h-chassis_z/2}" rpy="-1.5707 0.0 0.0"/>
-        <axis xyz="0 0 -1"/>
-    </joint>
-        <!-- LINK -->
-    <link name="right_wheel">
-        <xacro:inertial_cylinder mass="${wheel_m}" radius="${wheel_r}" length="${wheel_l}">
-            <origin xyz="0.0 0 0" rpy="0 0 0"/>
-        </xacro:inertial_cylinder>
-        <!-- <xacro:visual_cylinder radius="0.1" length="0.1" r="1" g="0" b="0" a="1">
-            <origin xyz="0.0 -0.3 0.1" rpy="-1.5707 0 0"/>
-        </xacro:visual_cylinder> -->
-        <visual>
-            <origin xyz="0.0 0 0" rpy="0 0 0"/>
-            <geometry>
-                <cylinder radius="${wheel_r}" length="${wheel_l}"/>
-            </geometry>
-            <material name="red">
-                <color rgba="1 0 0 1"/>
-            </material>
-        </visual>
-        <collision>
-            <origin xyz="0.0 0 0" rpy="0 0 0"/>
-            <geometry>
-                <cylinder radius="${wheel_r}" length="${wheel_l}"/>
-            </geometry>
-        </collision>
-    </link>
-    <!-- CASTER LINK -->
-    <joint name="caster_joint" type="fixed">
-        <parent link="chassis"/>
-        <child link="caster"/>
-        <origin xyz="${chassis_x/4} 0.0 ${caster_r-chassis_h-chassis_z/2}" rpy="0 0 0"/>
-    </joint>
-        <!-- LINK -->
-    <link name="caster">
-        <xacro:inertial_sphere mass="${caster_m}" radius="${caster_r}">
-            <origin xyz="0.0 0.0 0" rpy="0 0 0"/>
-        </xacro:inertial_sphere>
-        <!-- <xacro:visual_sphere radius="0.1" r="1" g="1" b="1" a="1" >
-            <origin xyz="0.5 0.0 0.1" rpy="0 0 0"/>
-        </xacro:visual_sphere> -->
-        <visual>
-            <origin xyz="0 0.0 0" rpy="0 0 0"/>
-            <geometry>
-                <sphere radius="${caster_r}"/>
-            </geometry>
-            <material name="black">
-                <color rgba="0 0 0 1"/>
-            </material>
-        </visual>
-        <collision>
-            <origin xyz="0 0.0 0" rpy="0 0 0"/>
-            <geometry>
-                <sphere radius="${caster_r}"/>
-            </geometry>
-        </collision>
-    </link>
-    <!-- FORK LINK -->
-    <joint name="fork_joint" type="fixed">
-        <parent link="chassis"/>
-        <child link="fork"/>
-        <origin xyz="${chassis_x/2+fork_x/2} 0.0 ${fork_z/2-chassis_z/2}" rpy="0.0 0.0 0.0"/>
-    </joint>
-        <!-- LINK -->
-    <link name="fork">
-        <xacro:inertial_box mass="${fork_m}" x="${fork_x}" y="${fork_y}" z="${fork_z}">
-            <origin xyz="0.0 0.0 0.0" rpy="0 0 0"/>
-        </xacro:inertial_box>
-        <!-- <xacro:visual_box  x="0.4" y="0.45" z="0.01" r="1" g="1" b="0" a="1">
-            <origin xyz="0.0 0.0 0.0  " rpy="0 0 0"/>
-        </xacro:visual_box> -->
-        <visual>
-            <origin xyz="0.0 0 0" rpy="0 0 0"/>
-            <geometry>
-                <box size="${fork_x} ${fork_y} ${fork_z}"/>
-            </geometry>
-            <material name="grey">
-                <color rgba="0.63 0.63 0.63 1"/>
-            </material>
-        </visual>
-        <collision>
-            <origin xyz="0.0 0 0" rpy="0 0 0"/>
-            <geometry>
-                <box size="${fork_x} ${fork_y} ${fork_z}"/>
-            </geometry>
-        </collision>
-    </link>
-    <gazebo reference="chassis">
-        <material>Gazebo/SkyBlue</material>
-    </gazebo>
-    <gazebo reference="left_wheel">
-        <material>Gazebo/Red</material>
-    </gazebo>
-    <gazebo reference="right_wheel">
-        <material>Gazebo/Red</material>
-    </gazebo>
-    <gazebo reference="fork">
-        <material>Gazebo/Grey</material>
-    </gazebo>
-    <gazebo reference="caster">
-        <material>Gazebo/Black</material>
-        <mu1 value="0.001"/>
-        <mu2 value="0.001"/>
-    </gazebo>
-</robot>
+/home/kuljot/Project/ball_follower/src/bot/description/robot_core.xacro

File: install/ball_follower/share/ball_follower/description/visual_macros.xacro (robot description, xacro)
@@ -1,56 +1 @@
-<?xml version="1.0"?>
-<robot xmlns:xacro="http://www.ros.org/wiki/xacro" >
-    <!-- Specify some standard visual calculations https://en.wikipedia.org/wiki/List_of_moments_of_inertia -->
-    <!-- These make use of xacro's mathematical functionality -->
-    <xacro:macro name="visual_box" params="x y z r g b a *origin">
-        <visual>
-            <xacro:insert_block name="origin"/>
-            <geometry>
-                <box size="${x} ${y} ${z}"/>
-            </geometry>
-            <material name="green">
-                <color rgba="${r} ${g} ${b} ${a}"/>
-            </material>
-        </visual>
-        <collision>
-            <xacro:insert_block name="origin"/>
-            <geometry>
-                <box size="${x} ${y} ${z}"/>
-            </geometry>
-        </collision>
-    </xacro:macro>
-    <xacro:macro name="visual_cylinder" params="length radius r g b a *origin">
-        <visual>
-            <xacro:insert_block name="origin"/>
-            <geometry>
-                <cylinder radius="${radius}" length="${length}"/>
-            </geometry>
-            <material name="red">
-                <color rgba="${r} ${g} ${b} ${a}"/>
-            </material>
-        </visual>
-        <collision>
-            <!-- <xacro:insert_block name="origin"/> -->
-            <geometry>
-                <cylinder radius="${radius}" length="${length}"/>
-            </geometry>
-        </collision>
-    </xacro:macro>
-    <xacro:macro name="visual_sphere" params="radius r g b a *origin">
-        <visual>
-            <xacro:insert_block name="origin"/>
-            <geometry>
-                <sphere radius="${radius}"/>
-            </geometry>
-            <material name="black">
-                <color rgba="${r} ${g} ${b} ${a}"/>
-            </material>
-        </visual>
-        <collision>
-            <xacro:insert_block name="origin"/>
-            <geometry>
-                <sphere radius="${radius}"/>
-            </geometry>
-        </collision>
-    </xacro:macro>
-</robot>
+/home/kuljot/Project/ball_follower/src/bot/description/visual_macros.xacro
